File: wiring/wiring.kicad_sch (KiCad schematic)
At the start: 16 parts, among them J1 Conn_01x03_Pin, J2 Motherboard_SVI2_SVD, J3 Motherboard_SVI2_SVC, J4 Motherboard_ATX_Reset, J5 Motherboard_ATX_Power_On, J6 Logic analyzer, SW1 SW_DIP_x01, U1 TXS0108EPW, U2 1117-1.8, U3 Motherboard SPI Flash, U4 LVC07A

Commit message: Fixed: Missing caps in schematic
Parts:
- added C3, C4: 10uF, symbol Device:C
Connections:
- net +3.3V: now also C3.1
- net GND: now also C3.2, C4.2
- net at SW1.1, U2.2 (VO): now also C4.1
